File: board/rj11_pi/rj11_pi.kicad_pcb (KiCad board)
At the start: 2 copper layers, 31.1 x 55.9 mm, 8 parts, among them J1 6P6C, J2 Conn_02x20_Odd_Even, Q1 Q_NPN_EBC, Q2 Q_NPN_EBC

Commit message: changed logging to print only when changed updated pins to work with pcb
Routing:
- net Net-(J2-Pad16): track 27.6 -> 31.6 mm
- net Net-(J1-Pad2): track 13.6 -> 13.1 mm
